File: geartrain-board/geartrain-board.sch (KiCad schematic (older format))
At the start: 196 parts

Commit message: Added strapping pin control to schematic
Parts:
- added R? (x2): 4.7k, symbol Device:R
- added SW?: DOWNLOAD BOOT, symbol Switch:SW_Push_DPDT
Connections:
- net +3V3: now also J?.3 (Pin_3); no longer J?.1 (Pin_1)
- net FPGA-TCK: now also J?.6 (Pin_6); no longer J?.4 (Pin_4)
- net FPGA-TDI: now also J?.4 (Pin_4); no longer J?.6 (Pin_6)
- net FPGA-TMS: now also J?.2 (Pin_2); no longer J?.3 (Pin_3)
- net GND: now also J?.1 (Pin_1), SW?.3 (C), SW?.6 (C); no longer J?.2 (Pin_2)
- net at U?.22 (GPIO2): now also R?.2
- net at U?.23 (GPIO0): now also R?.2
- new net: R?.1, SW?.2 (B)
- new net: R?.1, SW?.5 (B)
Other:
- note added: "DON'T CARE NOT USING SDIO FOLLOWER"
- note added: "GPIO0"
- note added: "GPIO2"
- note added: "GPIO5"
- note added: "MTDI"
- note added: "MTDO"
- note added: "PULL DOWN FOR UART FIRMWARE DOWNLOAD"
- note added: "PULL DOWN WITH GPIO0 TO DO UART FIRMWARE DOWNLOAD"
- note added: "PULL DOWN/LEAVE UNCONNECTED - 3.3V OPERATION"
- note added: "PULL UP/LEAVE UNCONNECTED - UART0 ACTIVE ON BOOT"
- note added: "STRAPPING PINS"
Changed lines of the file:
@@
 $EndComp
 Wire Wire Line
-	21000 8750 21050 8750
-Wire Wire Line
-	21000 8850 21050 8850
-Wire Wire Line
-	21000 8950 21150 8950
+	21000 8950 21500 8950
+Wire Wire Line
+	21000 8750 21500 8750
+Wire Wire Line
+	21000 8850 21150 8850
+Wire Wire Line
+	21000 9250 21150 9250
+Wire Wire Line
+	21000 9150 21150 9150
 Wire Wire Line
 	21000 9050 21150 9050
-Wire Wire Line
-	21000 9150 21150 9150
-Wire Wire Line
-	21000 9250 21150 9250
 $Comp
 L power:+3.3V #PWR?
 U 1 1 633FD834
-P 21050 8750
-F 0 "#PWR?" H 21050 8600 50  0001 C CNN
-F 1 "+3.3V" V 21065 8878 50  0000 L CNN
-F 2 "" H 21050 8750 50  0001 C CNN
-F 3 "" H 21050 8750 50  0001 C CNN
-	1    21050 8750
+P 21500 8950
+F 0 "#PWR?" H 21500 8800 50  0001 C CNN
+F 1 "+3.3V" V 21515 9078 50  0000 L CNN
+F 2 "" H 21500 8950 50  0001 C CNN
+F 3 "" H 21500 8950 50  0001 C CNN
+	1    21500 8950
 	0    1    1    0
 $EndComp
@@
 L power:GND #PWR?
 U 1 1 633FF1A2
-P 21050 8850
-F 0 "#PWR?" H 21050 8600 50  0001 C CNN
-F 1 "GND" V 21055 8722 50  0000 R CNN
-F 2 "" H 21050 8850 50  0001 C CNN
-F 3 "" H 21050 8850 50  0001 C CNN
-	1    21050 8850
+P 21500 8750
+F 0 "#PWR?" H 21500 8500 50  0001 C CNN
+F 1 "GND" V 21505 8622 50  0000 R CNN
+F 2 "" H 21500 8750 50  0001 C CNN
+F 3 "" H 21500 8750 50  0001 C CNN
+	1    21500 8750
 	0    -1   -1   0
 $EndComp
-Text Label 21150 8950 0    50   ~ 0
+Text Label 21150 8850 0    50   ~ 0
 FPGA-TMS
-Text Label 21150 9050 0    50   ~ 0
+Text Label 21150 9250 0    50   ~ 0
 FPGA-TCK
 Text Label 21150 9150 0    50   ~ 0
 FPGA-TDO
-Text Label 21150 9250 0    50   ~ 0
+Text Label 21150 9050 0    50   ~ 0
 FPGA-TDI
 $Comp
@@
 Text Notes 13950 2850 0    50   ~ 0
 FPGA CONTROL
-Connection ~ 16250 7000
+Text Notes 900  4700 0    50   ~ 0
+STRAPPING PINS
+Text Notes 1450 4850 0    50   ~ 0
+PULL DOWN/LEAVE UNCONNECTED - 3.3V OPERATION
+Text Notes 1450 4950 0    50   ~ 0
+PULL UP/LEAVE UNCONNECTED - UART0 ACTIVE ON BOOT
+Wire Wire Line
+	7350 5400 7450 5400
+Wire Wire Line
+	7450 5400 7450 5200
+$Comp
+L Switch:SW_Push_DPDT SW?
+U 1 1 61A94D3F
+P 7650 4650
+F 0 "SW?" V 7696 4262 50  0000 R CNN
+F 1 "DOWNLOAD BOOT" V 7605 4262 50  0000 R CNN
+F 2 "" H 7650 4850 50  0001 C CNN
+F 3 "~" H 7650 4850 50  0001 C CNN
+	1    7650 4650
+	0    -1   -1   0
+$EndComp
+Wire Wire Line
+	7350 5500 7850 5500
+Wire Wire Line
+	7850 5500 7850 5200
+$Comp
+L Device:R R?
+U 1 1 61BDE591
+P 7450 5050
+F 0 "R?" V 7400 4850 50  0000 C CNN
+F 1 "4.7k" V 7400 5250 50  0000 C CNN
+F 2 "" V 7380 5050 50  0001 C CNN
+F 3 "~" H 7450 5050 50  0001 C CNN
+	1    7450 5050
+	1    0    0    -1
+$EndComp
+Wire Wire Line
+	7450 4900 7450 4850
+$Comp
+L Device:R R?
+U 1 1 61BE7888
+P 7850 5050
+F 0 "R?" V 7800 4850 50  0000 C CNN
+F 1 "4.7k" V 7800 5250 50  0000 C CNN
+F 2 "" V 7780 5050 50  0001 C CNN
+F 3 "~" H 7850 5050 50  0001 C CNN
+	1    7850 5050
+	1    0    0    -1
+$EndComp
+Wire Wire Line
+	7850 4900 7850 4850
+$Comp
+L power:GND #PWR?
+U 1 1 61BE85C4
+P 8050 4300
+F 0 "#PWR?" H 8050 4050 50  0001 C CNN
+F 1 "GND" H 8055 4127 50  0000 C CNN
+F 2 "" H 8050 4300 50  0001 C CNN
+F 3 "" H 8050 4300 50  0001 C CNN
+	1    8050 4300
+	0    -1   -1   0
+$EndComp
+Wire Wire Line
+	7550 4450 7550 4300
+Wire Wire Line
+	7550 4300 7950 4300
+Wire Wire Line
+	7950 4450 7950 4300
+Connection ~ 7950 4300
+Wire Wire Line
+	7950 4300 8050 4300
+Text Notes 900  4850 0    50   ~ 0
+MTDI
+Text Notes 900  4950 0    50   ~ 0
+MTDO
+Text Notes 900  5050 0    50   ~ 0
+GPIO0
+Text Notes 1450 5050 0    50   ~ 0
+PULL DOWN FOR UART FIRMWARE DOWNLOAD
+Text Notes 900  5150 0    50   ~ 0
+GPIO2
+Text Notes 1450 5150 0    50   ~ 0
+PULL DOWN WITH GPIO0 TO DO UART FIRMWARE DOWNLOAD
+Text Notes 900  5250 0    50   ~ 0
+GPIO5
+Text Notes 1450 5250 0    50   ~ 0
+DON'T CARE NOT USING SDIO FOLLOWER
+Wire Notes Line style solid
+	850  4600 3750 4600
+Wire Notes Line style solid
+	3750 4600 3750 5300
+Wire Notes Line style solid
+	3750 5300 850  5300
+Wire Notes Line style solid
+	850  4600 850  5300
+Wire Notes Line
+	900  4700 1550 4700
 $EndSCHEMATC
